File: 3_Technical_Documents/PCB/PM3_Audio_and_DMX_Template/PM3_Audio_and_DMX_Template/Selection_VolCTRL.kicad_sch (KiCad schematic)
At the start: 2 parts, among them SW2 SW_DPDT_x2

Commit message: new push
Parts:
- renumbered RV4 to RV1, SW2 to SW3
Changed lines of the file:
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@@
 		(dnp no)
 		(fields_autoplaced yes)
-		(property "Reference" "#PWR042"
+		(property "Reference" "#PWR035"
 			(at 167.64 104.14 0)
 			(effects
@@
 			(project "PM3_Audio_and_DMX"
 				(path "/1f276d59-ad9b-4e70-a842-f3b7e562eb9b/2329d9ea-d5d7-4913-84c5-e85a54af032e/27da7c64-c1ae-436f-a80b-6f0a9911f136"
-					(reference "#PWR042")
+					(reference "#PWR035")
 					(unit 1)
 				)
@@
 		(on_board yes)
 		(dnp no)
-		(property "Reference" "RV4"
+		(property "Reference" "RV1"
 			(at 169.164 117.094 90)
 			(effects
@@
 			(project "PM3_Audio_and_DMX"
 				(path "/1f276d59-ad9b-4e70-a842-f3b7e562eb9b/2329d9ea-d5d7-4913-84c5-e85a54af032e/27da7c64-c1ae-436f-a80b-6f0a9911f136"
-					(reference "RV4")
+					(reference "RV1")
 					(unit 1)
 				)
@@
 		(on_board yes)
 		(dnp no)
-		(property "Reference" "#PWR021"
+		(property "Reference" "#PWR034"
 			(at 114.3 102.87 0)
 			(effects
@@
 			(project "PM3_Audio_and_DMX"
 				(path "/1f276d59-ad9b-4e70-a842-f3b7e562eb9b/2329d9ea-d5d7-4913-84c5-e85a54af032e/27da7c64-c1ae-436f-a80b-6f0a9911f136"
-					(reference "#PWR021")
+					(reference "#PWR034")
 					(unit 1)
 				)
@@
 		(dnp no)
 		(fields_autoplaced yes)
-		(property "Reference" "#PWR043"
+		(property "Reference" "#PWR036"
 			(at 167.64 116.84 0)
 			(effects
@@
 			(project "PM3_Audio_and_DMX"
 				(path "/1f276d59-ad9b-4e70-a842-f3b7e562eb9b/2329d9ea-d5d7-4913-84c5-e85a54af032e/27da7c64-c1ae-436f-a80b-6f0a9911f136"
-					(reference "#PWR043")
+					(reference "#PWR036")
 					(unit 1)
 				)
@@
 		(on_board yes)
 		(dnp no)
-		(property "Reference" "SW2"
+		(property "Reference" "SW3"
 			(at 121.92 102.87 0)
 			(effects
@@
 			(project "PM3_Audio_and_DMX"
 				(path "/1f276d59-ad9b-4e70-a842-f3b7e562eb9b/2329d9ea-d5d7-4913-84c5-e85a54af032e/27da7c64-c1ae-436f-a80b-6f0a9911f136"
-					(reference "SW2")
+					(reference "SW3")
 					(unit 2)
 				)
@@
 		(on_board yes)
 		(dnp no)
-		(property "Reference" "SW2"
+		(property "Reference" "SW3"
 			(at 123.698 100.33 0)
 			(effects
@@
 			(project "PM3_Audio_and_DMX"
 				(path "/1f276d59-ad9b-4e70-a842-f3b7e562eb9b/2329d9ea-d5d7-4913-84c5-e85a54af032e/27da7c64-c1ae-436f-a80b-6f0a9911f136"
-					(reference "SW2")
+					(reference "SW3")
 					(unit 1)
 				)
