File: 3_Technical_Documents/PCB/PM3_Audio_and_DMX_Template/PM3_Audio_and_DMX_Template/digital_power_supply.kicad_sch (KiCad schematic)
At the start: 7 parts, among them U8 LT3045xMSE

Commit message: new push
Parts:
- renumbered C88 to C10, C29 to C7, C90 to C8, C28 to C9, R57 to R6, R58 to R7, U8 to U2
Changed lines of the file:
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@@
 		(dnp no)
 		(fields_autoplaced yes)
-		(property "Reference" "C28"
+		(property "Reference" "C9"
 			(at 119.38 96.5199 0)
 			(effects
@@
 			(project "PM3_Audio_and_DMX"
 				(path "/1f276d59-ad9b-4e70-a842-f3b7e562eb9b/0cd82055-ce21-4aed-acf2-771a9b05e7c5/7ea0a49e-7c2f-4e20-9587-1e84a77cfe1f"
-					(reference "C28")
+					(reference "C9")
 					(unit 1)
 				)
@@
 		(dnp no)
 		(fields_autoplaced yes)
-		(property "Reference" "#PWR060"
+		(property "Reference" "#PWR027"
 			(at 101.6 87.63 0)
 			(effects
@@
 			(project "PM3_Audio_and_DMX"
 				(path "/1f276d59-ad9b-4e70-a842-f3b7e562eb9b/0cd82055-ce21-4aed-acf2-771a9b05e7c5/7ea0a49e-7c2f-4e20-9587-1e84a77cfe1f"
-					(reference "#PWR060")
-					(unit 1)
-				)
-				(path "/1f276d59-ad9b-4e70-a842-f3b7e562eb9b/2329d9ea-d5d7-4913-84c5-e85a54af032e/4134625c-b4ab-48ae-8ee9-d10f38bbf1f1"
-					(reference "#PWR060")
+					(reference "#PWR027")
+					(unit 1)
+				)
+				(path "/1f276d59-ad9b-4e70-a842-f3b7e562eb9b/2329d9ea-d5d7-4913-84c5-e85a54af032e/4134625c-b4ab-48ae-8ee9-d10f38bbf1f1"
+					(reference "#PWR066")
 					(unit 1)
 				)
@@
 		(dnp no)
 		(fields_autoplaced yes)
-		(property "Reference" "U8"
+		(property "Reference" "U2"
 			(at 143.51 73.66 0)
 			(effects
@@
 			(project "PM3_Audio_and_DMX"
 				(path "/1f276d59-ad9b-4e70-a842-f3b7e562eb9b/0cd82055-ce21-4aed-acf2-771a9b05e7c5/7ea0a49e-7c2f-4e20-9587-1e84a77cfe1f"
-					(reference "U8")
-					(unit 1)
-				)
-				(path "/1f276d59-ad9b-4e70-a842-f3b7e562eb9b/2329d9ea-d5d7-4913-84c5-e85a54af032e/4134625c-b4ab-48ae-8ee9-d10f38bbf1f1"
-					(reference "U8")
+					(reference "U2")
+					(unit 1)
+				)
+				(path "/1f276d59-ad9b-4e70-a842-f3b7e562eb9b/2329d9ea-d5d7-4913-84c5-e85a54af032e/4134625c-b4ab-48ae-8ee9-d10f38bbf1f1"
+					(reference "U9")
 					(unit 1)
 				)
@@
 		(dnp no)
 		(fields_autoplaced yes)
-		(property "Reference" "#PWR0113"
+		(property "Reference" "#PWR028"
 			(at 114.3 87.63 0)
 			(effects
@@
 			(project "PM3_Audio_and_DMX"
 				(path "/1f276d59-ad9b-4e70-a842-f3b7e562eb9b/0cd82055-ce21-4aed-acf2-771a9b05e7c5/7ea0a49e-7c2f-4e20-9587-1e84a77cfe1f"
-					(reference "#PWR0113")
-					(unit 1)
-				)
-				(path "/1f276d59-ad9b-4e70-a842-f3b7e562eb9b/2329d9ea-d5d7-4913-84c5-e85a54af032e/4134625c-b4ab-48ae-8ee9-d10f38bbf1f1"
-					(reference "#PWR0115")
+					(reference "#PWR028")
+					(unit 1)
+				)
+				(path "/1f276d59-ad9b-4e70-a842-f3b7e562eb9b/2329d9ea-d5d7-4913-84c5-e85a54af032e/4134625c-b4ab-48ae-8ee9-d10f38bbf1f1"
+					(reference "#PWR067")
 					(unit 1)
 				)
@@
 		(dnp no)
 		(fields_autoplaced yes)
-		(property "Reference" "R57"
+		(property "Reference" "R6"
 			(at 133.35 96.5199 0)
 			(effects
@@
 			(project "PM3_Audio_and_DMX"
 				(path "/1f276d59-ad9b-4e70-a842-f3b7e562eb9b/0cd82055-ce21-4aed-acf2-771a9b05e7c5/7ea0a49e-7c2f-4e20-9587-1e84a77cfe1f"
-					(reference "R57")
-					(unit 1)
-				)
-				(path "/1f276d59-ad9b-4e70-a842-f3b7e562eb9b/2329d9ea-d5d7-4913-84c5-e85a54af032e/4134625c-b4ab-48ae-8ee9-d10f38bbf1f1"
-					(reference "R57")
+					(reference "R6")
+					(unit 1)
+				)
+				(path "/1f276d59-ad9b-4e70-a842-f3b7e562eb9b/2329d9ea-d5d7-4913-84c5-e85a54af032e/4134625c-b4ab-48ae-8ee9-d10f38bbf1f1"
+					(reference "R27")
 					(unit 1)
 				)
@@
 		(dnp no)
 		(fields_autoplaced yes)
-		(property "Reference" "C88"
+		(property "Reference" "C10"
 			(at 173.99 87.6299 0)
 			(effects
@@
 			(project "PM3_Audio_and_DMX"
 				(path "/1f276d59-ad9b-4e70-a842-f3b7e562eb9b/0cd82055-ce21-4aed-acf2-771a9b05e7c5/7ea0a49e-7c2f-4e20-9587-1e84a77cfe1f"
-					(reference "C88")
-					(unit 1)
-				)
-				(path "/1f276d59-ad9b-4e70-a842-f3b7e562eb9b/2329d9ea-d5d7-4913-84c5-e85a54af032e/4134625c-b4ab-48ae-8ee9-d10f38bbf1f1"
-					(reference "C88")
+					(reference "C10")
+					(unit 1)
+				)
+				(path "/1f276d59-ad9b-4e70-a842-f3b7e562eb9b/2329d9ea-d5d7-4913-84c5-e85a54af032e/4134625c-b4ab-48ae-8ee9-d10f38bbf1f1"
+					(reference "C29")
 					(unit 1)
 				)
@@
 		(dnp no)
 		(fields_autoplaced yes)
-		(property "Reference" "#PWR061"
+		(property "Reference" "#PWR030"
 			(at 130.81 116.84 0)
 			(effects
@@
 			(project "PM3_Audio_and_DMX"
 				(path "/1f276d59-ad9b-4e70-a842-f3b7e562eb9b/0cd82055-ce21-4aed-acf2-771a9b05e7c5/7ea0a49e-7c2f-4e20-9587-1e84a77cfe1f"
-					(reference "#PWR061")
-					(unit 1)
-				)
-				(path "/1f276d59-ad9b-4e70-a842-f3b7e562eb9b/2329d9ea-d5d7-4913-84c5-e85a54af032e/4134625c-b4ab-48ae-8ee9-d10f38bbf1f1"
-					(reference "#PWR061")
+					(reference "#PWR030")
+					(unit 1)
+				)
+				(path "/1f276d59-ad9b-4e70-a842-f3b7e562eb9b/2329d9ea-d5d7-4913-84c5-e85a54af032e/4134625c-b4ab-48ae-8ee9-d10f38bbf1f1"
+					(reference "#PWR069")
 					(unit 1)
 				)
@@
 		(on_board yes)
 		(dnp no)
-		(property "Reference" "R58"
+		(property "Reference" "R7"
 			(at 149.86 71.12 0)
 			(effects
@@
 			(project "PM3_Audio_and_DMX"
 				(path "/1f276d59-ad9b-4e70-a842-f3b7e562eb9b/0cd82055-ce21-4aed-acf2-771a9b05e7c5/7ea0a49e-7c2f-4e20-9587-1e84a77cfe1f"
-					(reference "R58")
-					(unit 1)
-				)
-				(path "/1f276d59-ad9b-4e70-a842-f3b7e562eb9b/2329d9ea-d5d7-4913-84c5-e85a54af032e/4134625c-b4ab-48ae-8ee9-d10f38bbf1f1"
-					(reference "R58")
+					(reference "R7")
+					(unit 1)
+				)
+				(path "/1f276d59-ad9b-4e70-a842-f3b7e562eb9b/2329d9ea-d5d7-4913-84c5-e85a54af032e/4134625c-b4ab-48ae-8ee9-d10f38bbf1f1"
+					(reference "R28")
 					(unit 1)
 				)
@@
 		(dnp no)
 		(fields_autoplaced yes)
-		(property "Reference" "#PWR0110"
+		(property "Reference" "#PWR031"
 			(at 143.51 104.14 0)
 			(effects
@@
 			(project "PM3_Audio_and_DMX"
 				(path "/1f276d59-ad9b-4e70-a842-f3b7e562eb9b/0cd82055-ce21-4aed-acf2-771a9b05e7c5/7ea0a49e-7c2f-4e20-9587-1e84a77cfe1f"
-					(reference "#PWR0110")
-					(unit 1)
-				)
-				(path "/1f276d59-ad9b-4e70-a842-f3b7e562eb9b/2329d9ea-d5d7-4913-84c5-e85a54af032e/4134625c-b4ab-48ae-8ee9-d10f38bbf1f1"
-					(reference "#PWR0110")
+					(reference "#PWR031")
+					(unit 1)
+				)
+				(path "/1f276d59-ad9b-4e70-a842-f3b7e562eb9b/2329d9ea-d5d7-4913-84c5-e85a54af032e/4134625c-b4ab-48ae-8ee9-d10f38bbf1f1"
+					(reference "#PWR070")
 					(unit 1)
 				)
@@
 		(dnp no)
 		(fields_autoplaced yes)
-		(property "Reference" "#PWR0109"
+		(property "Reference" "#PWR029"
 			(at 120.65 86.36 0)
 			(effects
@@
 			(project "PM3_Audio_and_DMX"
 				(path "/1f276d59-ad9b-4e70-a842-f3b7e562eb9b/0cd82055-ce21-4aed-acf2-771a9b05e7c5/7ea0a49e-7c2f-4e20-9587-1e84a77cfe1f"
-					(reference "#PWR0109")
-					(unit 1)
-				)
-				(path "/1f276d59-ad9b-4e70-a842-f3b7e562eb9b/2329d9ea-d5d7-4913-84c5-e85a54af032e/4134625c-b4ab-48ae-8ee9-d10f38bbf1f1"
-					(reference "#PWR0109")
+					(reference "#PWR029")
+					(unit 1)
+				)
+				(path "/1f276d59-ad9b-4e70-a842-f3b7e562eb9b/2329d9ea-d5d7-4913-84c5-e85a54af032e/4134625c-b4ab-48ae-8ee9-d10f38bbf1f1"
+					(reference "#PWR068")
 					(unit 1)
 				)
@@
 		(on_board yes)
 		(dnp no)
-		(property "Reference" "C29"
+		(property "Reference" "C7"
 			(at 106.172 73.406 90)
 			(effects
@@
 			(project "PM3_Audio_and_DMX"
 				(path "/1f276d59-ad9b-4e70-a842-f3b7e562eb9b/0cd82055-ce21-4aed-acf2-771a9b05e7c5/7ea0a49e-7c2f-4e20-9587-1e84a77cfe1f"
-					(reference "C29")
-					(unit 1)
-				)
-				(path "/1f276d59-ad9b-4e70-a842-f3b7e562eb9b/2329d9ea-d5d7-4913-84c5-e85a54af032e/4134625c-b4ab-48ae-8ee9-d10f38bbf1f1"
-					(reference "C29")
+					(reference "C7")
+					(unit 1)
+				)
+				(path "/1f276d59-ad9b-4e70-a842-f3b7e562eb9b/2329d9ea-d5d7-4913-84c5-e85a54af032e/4134625c-b4ab-48ae-8ee9-d10f38bbf1f1"
+					(reference "C26")
 					(unit 1)
 				)
@@
 		(dnp no)
 		(fields_autoplaced yes)
-		(property "Reference" "#PWR0112"
+		(property "Reference" "#PWR032"
 			(at 170.18 102.87 0)
 			(effects
@@
 			(project "PM3_Audio_and_DMX"
 				(path "/1f276d59-ad9b-4e70-a842-f3b7e562eb9b/0cd82055-ce21-4aed-acf2-771a9b05e7c5/7ea0a49e-7c2f-4e20-9587-1e84a77cfe1f"
-					(reference "#PWR0112")
-					(unit 1)
-				)
-				(path "/1f276d59-ad9b-4e70-a842-f3b7e562eb9b/2329d9ea-d5d7-4913-84c5-e85a54af032e/4134625c-b4ab-48ae-8ee9-d10f38bbf1f1"
-					(reference "#PWR0112")
+					(reference "#PWR032")
+					(unit 1)
+				)
+				(path "/1f276d59-ad9b-4e70-a842-f3b7e562eb9b/2329d9ea-d5d7-4913-84c5-e85a54af032e/4134625c-b4ab-48ae-8ee9-d10f38bbf1f1"
+					(reference "#PWR071")
 					(unit 1)
 				)
@@
 		(dnp no)
 		(fields_autoplaced yes)
-		(property "Reference" "C90"
+		(property "Reference" "C8"
 			(at 118.11 72.3899 0)
 			(effects
@@
 			(project "PM3_Audio_and_DMX"
 				(path "/1f276d59-ad9b-4e70-a842-f3b7e562eb9b/0cd82055-ce21-4aed-acf2-771a9b05e7c5/7ea0a49e-7c2f-4e20-9587-1e84a77cfe1f"
-					(reference "C90")
-					(unit 1)
-				)
-				(path "/1f276d59-ad9b-4e70-a842-f3b7e562eb9b/2329d9ea-d5d7-4913-84c5-e85a54af032e/4134625c-b4ab-48ae-8ee9-d10f38bbf1f1"
-					(reference "C92")
-					(unit 1)
-				)
+					(reference "C8")
+					(unit 1)
+				)
+				(path "/1f276d59-ad9b-4e70-a842-f3b7e562eb9b/2329d9ea-d5d7-4913-84c5-e85a54af032e/4134625c-b4ab-48ae-8ee9-d10f38bbf1f1"
+					(reference "C27")
+					(unit 1)
+				)

Commit message: rework esp32, codec and layout
Parts:
- renumbered R6 to R5, R7 to R6
Changed lines of the file:
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@@
 				)
 				(path "/1f276d59-ad9b-4e70-a842-f3b7e562eb9b/2329d9ea-d5d7-4913-84c5-e85a54af032e/4134625c-b4ab-48ae-8ee9-d10f38bbf1f1"
-					(reference "#PWR066")
+					(reference "#PWR065")
 					(unit 1)
 				)
@@
 				)
 				(path "/1f276d59-ad9b-4e70-a842-f3b7e562eb9b/2329d9ea-d5d7-4913-84c5-e85a54af032e/4134625c-b4ab-48ae-8ee9-d10f38bbf1f1"
-					(reference "#PWR067")
+					(reference "#PWR066")
 					(unit 1)
 				)
@@
 		(dnp no)
 		(fields_autoplaced yes)
-		(property "Reference" "R6"
+		(property "Reference" "R5"
 			(at 133.35 96.5199 0)
 			(effects
@@
 			(project "PM3_Audio_and_DMX"
 				(path "/1f276d59-ad9b-4e70-a842-f3b7e562eb9b/0cd82055-ce21-4aed-acf2-771a9b05e7c5/7ea0a49e-7c2f-4e20-9587-1e84a77cfe1f"
-					(reference "R6")
-					(unit 1)
-				)
-				(path "/1f276d59-ad9b-4e70-a842-f3b7e562eb9b/2329d9ea-d5d7-4913-84c5-e85a54af032e/4134625c-b4ab-48ae-8ee9-d10f38bbf1f1"
-					(reference "R27")
+					(reference "R5")
+					(unit 1)
+				)
+				(path "/1f276d59-ad9b-4e70-a842-f3b7e562eb9b/2329d9ea-d5d7-4913-84c5-e85a54af032e/4134625c-b4ab-48ae-8ee9-d10f38bbf1f1"
+					(reference "R26")
 					(unit 1)
 				)
@@
 				)
 				(path "/1f276d59-ad9b-4e70-a842-f3b7e562eb9b/2329d9ea-d5d7-4913-84c5-e85a54af032e/4134625c-b4ab-48ae-8ee9-d10f38bbf1f1"
-					(reference "#PWR069")
+					(reference "#PWR068")
 					(unit 1)
 				)
@@
 		(on_board yes)
 		(dnp no)
-		(property "Reference" "R7"
+		(property "Reference" "R6"
 			(at 149.86 71.12 0)
 			(effects
@@
 			(project "PM3_Audio_and_DMX"
 				(path "/1f276d59-ad9b-4e70-a842-f3b7e562eb9b/0cd82055-ce21-4aed-acf2-771a9b05e7c5/7ea0a49e-7c2f-4e20-9587-1e84a77cfe1f"
-					(reference "R7")
-					(unit 1)
-				)
-				(path "/1f276d59-ad9b-4e70-a842-f3b7e562eb9b/2329d9ea-d5d7-4913-84c5-e85a54af032e/4134625c-b4ab-48ae-8ee9-d10f38bbf1f1"
-					(reference "R28")
+					(reference "R6")
+					(unit 1)
+				)
+				(path "/1f276d59-ad9b-4e70-a842-f3b7e562eb9b/2329d9ea-d5d7-4913-84c5-e85a54af032e/4134625c-b4ab-48ae-8ee9-d10f38bbf1f1"
+					(reference "R27")
 					(unit 1)
 				)
@@
 				)
 				(path "/1f276d59-ad9b-4e70-a842-f3b7e562eb9b/2329d9ea-d5d7-4913-84c5-e85a54af032e/4134625c-b4ab-48ae-8ee9-d10f38bbf1f1"
-					(reference "#PWR070")
+					(reference "#PWR069")
 					(unit 1)
 				)
@@
 				)
 				(path "/1f276d59-ad9b-4e70-a842-f3b7e562eb9b/2329d9ea-d5d7-4913-84c5-e85a54af032e/4134625c-b4ab-48ae-8ee9-d10f38bbf1f1"
-					(reference "#PWR068")
+					(reference "#PWR067")
 					(unit 1)
 				)
@@
 				)
 				(path "/1f276d59-ad9b-4e70-a842-f3b7e562eb9b/2329d9ea-d5d7-4913-84c5-e85a54af032e/4134625c-b4ab-48ae-8ee9-d10f38bbf1f1"
-					(reference "#PWR071")
-					(unit 1)
-				)
+					(reference "#PWR070")
+					(unit 1)
+				)
