File: 3_Technical_Documents/PCB/PM3_Audio_and_DMX_Template/PM3_Audio_and_DMX_Template/pm3_audio.kicad_sch (KiCad schematic)
At the start: 10 parts, among them J2 LINE_IN, J3 LINE_OUT, J4 HEADPHONE_JACK

Commit message: new push
Parts:
- removed RV1: 50k, Potentiometer_THT:Potentiometer_Bourns_PTV09A-1_Single_Vertical, symbol Device:R_Potentiometer
- removed RV3: 50k stereo, Potentiometer_THT:Potentiometer_Bourns_PTV112-4_Dual_Vertical, symbol Device:R_Potentiometer_Dual
- renumbered J4 to J3, J3 to J4, R10 to R14, TP8 to TP6, TP9 to TP7, TP12 to TP8, TP13 to TP9

Commit message: rework esp32, codec and layout
Parts:
- renumbered R14 to R13
Changed lines of the file:
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@@
 		(dnp no)
 		(fields_autoplaced yes)
-		(property "Reference" "R14"
+		(property "Reference" "R13"
 			(at 60.96 41.9099 0)
 			(effects
@@
 			(project ""
 				(path "/1f276d59-ad9b-4e70-a842-f3b7e562eb9b/2329d9ea-d5d7-4913-84c5-e85a54af032e"
-					(reference "R14")
+					(reference "R13")
 					(unit 1)
 				)
@@
 		(dnp no)
 		(fields_autoplaced yes)
-		(property "Reference" "#PWR046"
+		(property "Reference" "#PWR045"
 			(at 260.35 147.32 0)
 			(effects
@@
 			(project "PM3_Audio_and_DMX"
 				(path "/1f276d59-ad9b-4e70-a842-f3b7e562eb9b/2329d9ea-d5d7-4913-84c5-e85a54af032e"
-					(reference "#PWR046")
+					(reference "#PWR045")
 					(unit 1)
 				)
@@
 		(dnp no)
 		(fields_autoplaced yes)
-		(property "Reference" "#PWR040"
+		(property "Reference" "#PWR039"
 			(at 34.29 60.96 0)
 			(effects
@@
 			(project "PM3_Audio_and_DMX"
 				(path "/1f276d59-ad9b-4e70-a842-f3b7e562eb9b/2329d9ea-d5d7-4913-84c5-e85a54af032e"
-					(reference "#PWR040")
+					(reference "#PWR039")
 					(unit 1)
 				)
@@
 		(dnp no)
 		(fields_autoplaced yes)
-		(property "Reference" "#PWR042"
+		(property "Reference" "#PWR041"
 			(at 58.42 36.83 0)
 			(effects
@@
 			(project ""
 				(path "/1f276d59-ad9b-4e70-a842-f3b7e562eb9b/2329d9ea-d5d7-4913-84c5-e85a54af032e"
-					(reference "#PWR042")
+					(reference "#PWR041")
 					(unit 1)
 				)
@@
 		(dnp no)
 		(fields_autoplaced yes)
-		(property "Reference" "#PWR045"
+		(property "Reference" "#PWR044"
 			(at 260.35 120.65 0)
 			(effects
@@
 			(project "PM3_Audio_and_DMX"
 				(path "/1f276d59-ad9b-4e70-a842-f3b7e562eb9b/2329d9ea-d5d7-4913-84c5-e85a54af032e"
-					(reference "#PWR045")
+					(reference "#PWR044")
 					(unit 1)
 				)
@@
 		(dnp no)
 		(fields_autoplaced yes)
-		(property "Reference" "#PWR043"
+		(property "Reference" "#PWR042"
 			(at 124.46 52.07 0)
 			(effects
@@
 			(project ""
 				(path "/1f276d59-ad9b-4e70-a842-f3b7e562eb9b/2329d9ea-d5d7-4913-84c5-e85a54af032e"
-					(reference "#PWR043")
+					(reference "#PWR042")
 					(unit 1)
 				)
@@
 		(dnp no)
 		(fields_autoplaced yes)
-		(property "Reference" "#PWR041"
+		(property "Reference" "#PWR040"
 			(at 34.29 106.68 0)
 			(effects
@@
 			(project "PM3_Audio_and_DMX"
 				(path "/1f276d59-ad9b-4e70-a842-f3b7e562eb9b/2329d9ea-d5d7-4913-84c5-e85a54af032e"
-					(reference "#PWR041")
+					(reference "#PWR040")
 					(unit 1)
 				)
@@
 		(dnp no)
 		(fields_autoplaced yes)
-		(property "Reference" "#PWR044"
+		(property "Reference" "#PWR043"
 			(at 124.46 67.31 0)
 			(effects
@@
 			(project ""
 				(path "/1f276d59-ad9b-4e70-a842-f3b7e562eb9b/2329d9ea-d5d7-4913-84c5-e85a54af032e"
-					(reference "#PWR044")
-					(unit 1)
-				)
+					(reference "#PWR043")
+					(unit 1)
+				)
