File: 3_Technical_Documents/PCB/PM3_Audio_and_DMX_Template/PM3_Audio_and_DMX_Template/PM3_Audio_and_DMX.kicad_pcb (KiCad board)
At the start: 4 copper layers, 66 x 121.9 mm, 190 parts, among them J1 DMX-out, J2 LINE_IN, J3 HEADPHONE_JACK, J4 LINE_OUT, P1 Conn_02x32_Odd_Even, P2 Conn_02x32_Odd_Even, SW1 SW_Push, SW2 SW_Push, SW3 SW_DPDT_x2, U1 ESP32-WROOM-32E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

Commit message: layout fix
Parts:
- moved H3 100.0 mm to (191.8, 127.7), turned to 90 degrees
- moved H4 99.7 mm to (191.8, 71.8), turned to 90 degrees
- moved C16 97.2 mm to (195.6, 104.1), turned to -90 degrees
- moved MK1 96.0 mm to (194.9, 100.0), turned to 90 degrees
- moved TP10 96.0 mm to (194.2, 90.0), turned to -90 degrees
- moved C49 95.6 mm to (194.2, 107.1), turned to -90 degrees
- moved R17 95.0 mm to (194.0, 104.0), turned to -90 degrees
- moved U12 94.6 mm to (190.6, 120.0), turned to -90 degrees
- moved R41 94.5 mm to (192.1, 114.5), turned to 180 degrees
- moved C44 94.1 mm to (192.1, 113.0), turned to 180 degrees
- moved C14 93.0 mm to (192.3, 107.3), turned to 90 degrees
- moved R14 92.7 mm to (192.4, 95.7), turned to 90 degrees
- moved C45 92.3 mm to (192.1, 104.0), turned to 180 degrees
- moved R42 92.2 mm to (192.1, 102.5), turned to 180 degrees
- moved U6 91.4 mm to (191.5, 103.0), turned to 90 degrees
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Routing:
- net GND: vias 37 -> 31
Other:
- board size 66 x 121.9 mm -> 121.9 x 66 mm

Commit message: added 3d models
Other:
- board text added: "PM3-Audio / 2025 grebnbog & perritho"
- board text removed: "PM3-Audio & DMX Template (c) rost@zhaw.ch 09 /2025"
Changed lines of the file:
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@@
 		)
 		(embedded_fonts no)
-		(model "${KICAD9_3DMODEL_DIR}/Button_Switch_SMD.3dshapes/SW_DPDT_CK_JS202011JCQN.step"
+		(model "C:/Users/Thomas/Documents/git/PM3/3_Technical_Documents/PCB/libraries/switch/JS202011JCQN--3DModel-STEP-1.STEP"
 			(offset
 				(xyz 0 0 0)
@@
 			)
 			(rotate
-				(xyz 0 0 0)
+				(xyz -90 -0 -90)
 			)
 		)
@@
 		)
 		(embedded_fonts no)
-		(model "${KICAD9_3DMODEL_DIR}/Potentiometer_THT.3dshapes/Potentiometer_Bourns_PTV112-4_Dual_Vertical.step"
+		(model "C:/Users/Thomas/Documents/git/PM3/3_Technical_Documents/PCB/libraries/Potentiometer/PTV112-4420A-B503--3DModel-STEP-269445.STEP"
 			(offset
-				(xyz 0 0 0)
+				(xyz 11 -3 0)
 			)
 			(scale
@@
 			)
 			(rotate
-				(xyz 0 0 0)
+				(xyz -90 -0 90)
 			)
 		)
@@
 		)
 		(embedded_fonts no)
-		(model "${KICAD9_3DMODEL_DIR}/Connector_Audio.3dshapes/Jack_3.5mm_CUI_SJ-3523-SMT_Horizontal.step"
+		(model "C:/Users/Thomas/Documents/git/PM3/3_Technical_Documents/PCB/libraries/3m5 jack/SJ-3523-SMT-TR--3DModel-STEP-1.STEP"
 			(offset
-				(xyz 0 0 0)
+				(xyz 0 6 3)
 			)
 			(scale
@@
 			)
 			(rotate
-				(xyz 0 0 0)
+				(xyz -90 -0 -180)
 			)
 		)
@@
 		)
 		(embedded_fonts no)
-		(model "${KICAD9_3DMODEL_DIR}/Connector_Audio.3dshapes/Jack_3.5mm_CUI_SJ-3523-SMT_Horizontal.step"
+		(model "C:/Users/Thomas/Documents/git/PM3/3_Technical_Documents/PCB/libraries/3m5 jack/SJ-3523-SMT-TR--3DModel-STEP-1.STEP"
 			(offset
-				(xyz 0 0 0)
+				(xyz 0 6 3)
 			)
 			(scale
@@
 			)
 			(rotate
-				(xyz 0 0 0)
+				(xyz -90 -0 -180)
 			)
 		)
@@
 		)
 		(embedded_fonts no)
-		(model "${KICAD9_3DMODEL_DIR}/Connector_Audio.3dshapes/Jack_3.5mm_CUI_SJ-3523-SMT_Horizontal.step"
+		(model "C:/Users/Thomas/Documents/git/PM3/3_Technical_Documents/PCB/libraries/3m5 jack/SJ-3523-SMT-TR--3DModel-STEP-1.STEP"
 			(offset
-				(xyz 0 0 0)
+				(xyz 0 6 3)
 			)
 			(scale
@@
 			)
 			(rotate
-				(xyz 0 0 0)
+				(xyz -90 -0 -180)
 			)
 		)
@@
 		)
 		(embedded_fonts no)
-		(model "${KICAD9_3DMODEL_DIR}/Potentiometer_THT.3dshapes/Potentiometer_Bourns_PTV112-4_Dual_Vertical.step"
+		(model "C:/Users/Thomas/Documents/git/PM3/3_Technical_Documents/PCB/libraries/Potentiometer/PTV112-4420A-B503--3DModel-STEP-269445.STEP"
 			(offset
-				(xyz 0 0 0)
+				(xyz 11 -3 0)
 			)
 			(scale
@@
 			)
 			(rotate
-				(xyz 0 0 0)
+				(xyz -90 -0 90)
 			)
 		)
@@
 		)
 	)
-	(gr_text "PM3-Audio & DMX Template\n(c) rost@zhaw.ch 09\n/2025"
+	(gr_text "PM3-Audio / 2025\ngrebnbog & perritho\n"
 		(at 92.81 68.95 0)
 		(layer "F.SilkS")

Commit message: finalized design and generated gerber
Parts:
- added G***: LOGO, LOGO, F.Cu at (90.2, 100.0)
- added G***: LOGO, LOGO, B.Cu at (98.3, 97.1)
- added G***: LOGO, LOGO, B.Cu at (106.8, 110.5)
- moved C2 3.25 mm to (155.2, 69.8), turned to 180 degrees
- renumbered SW2 to BOOT1, SW1 to EN1
Routing:
- net GND: track 691.8 -> 667.0 mm, vias 31 -> 36
- net /PM3 Audio/Headphone Amplifier/in_r: track 59.6 -> 62.4 mm
- net /PM3 Audio/Codec with analog line buffers/Audio Output/AOUTB-: track 41.7 -> 39.8 mm
- net PA8: track 44.4 -> 42.6 mm
- net /PM3 Audio/Analog Power Supply/Power_in: track 39.8 -> 38.5 mm
- net PC9: track 44.9 -> 43.7 mm
- net VL: track 132.7 -> 133.8 mm
- net PE2: track 69.4 -> 68.3 mm
- net VA: track 221.0 -> 221.7 mm
- net Net-(U5-RO): track 2.78 -> 3.43 mm
- net /PM3 Audio/Codec with analog line buffers/Audio Output/AOUTB+: track 44.1 -> 43.6 mm
- added copper zone on In2.Cu, net GND
Other:
- board text added: "Analog Input"
- board text added: "Analog Output"
- board text added: "CODEC"
- board text added: "ESP POW"
- board text added: "IN"
- board text added: "Input Vol."
- board text added: "OUT"
- board text added: "Output Vol."
- board text added: "SELECT"

Commit message: reqorked pcb
Parts:
- added R64: 10k, Resistor_SMD:R_0603_1608Metric, F.Cu at (113.6, 95.4)
- C34, C35: moved to B.Cu
- moved C33 56.0 mm to (92.0, 88.8), turned to 90 degrees
- moved C32 55.8 mm to (93.9, 88.8), turned to 90 degrees
- moved C35 38.3 mm to (103.2, 95.8)
- moved C34 38.2 mm to (105.2, 95.8)
- moved C39 32.0 mm to (106.5, 83.4), turned to 0 degrees
- moved C36 31.4 mm to (106.4, 85.4), turned to 0 degrees
Connections:
- U10 pad 23: VL -> unconnected-(U10-~{AMUTEC}-Pad23)
- U10 pad 28: VL -> unconnected-(U10-~{BMUTEC}-Pad28)
Routing:
- net PB4: track 46.7 -> 49.7 mm
- net +5V: track 113.5 -> 116.5 mm
- net GND: track 667.0 -> 665.2 mm, vias 36 -> 39
- net VA: track 221.7 -> 223.3 mm
- net PC12: track 47.2 -> 45.6 mm
- net VD: track 45.1 -> 43.6 mm
- net VL: track 133.8 -> 134.4 mm
