File: 3_Technical_Documents/PCB/PM3_Audio_and_DMX_Template/PM3_Audio_and_DMX_Template/PM3_Audio_and_DMX.kicad_pcb (KiCad board)
At the start: 4 copper layers, 121.9 x 66 mm, 194 parts, among them J1 DMX-out, J2 LINE_IN, J3 HEADPHONE_JACK, J4 LINE_OUT, P1 Conn_02x32_Odd_Even, P2 Conn_02x32_Odd_Even, SW3 SW_DPDT_x2, U1 ESP32-WROOM-32E, U10 CS4271, U11 OPA2134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

Commit message: fixed pcb, again.
Parts:
- moved C33 0.10 mm to (91.9, 88.8)
Routing:
- net VCOM: track 121.5 -> 152.6 mm, vias 5 -> 4
- net VA: track 223.3 -> 250.4 mm
- net /PM3 Audio/Headphone Amplifier/in_l: track 54.6 -> 62.2 mm, vias 1 -> 2
- net /PM3 Audio/Codec with analog line buffers/LINE_OUT_L: track 86.0 -> 86.6 mm
- net GND: track 665.2 -> 665.6 mm, vias 39 -> 65
- net /PM3 Audio/Headphone Amplifier/in_r: track 62.4 -> 62.8 mm, vias 1 -> 3
- net DMX_GND: vias 4 -> 21

Commit message: final final
Parts:
- moved J2 1.20 mm to (178.5, 75.3)
- moved J4 1.20 mm to (167.0, 75.3)
- moved J3 0.90 mm to (83.6, 106.5)
Routing:
- net GND: track 665.6 -> 601.6 mm, vias 65 -> 67
- net /PM3 Audio/Codec with analog line buffers/LINE_OUT_R: track 86.1 -> 87.8 mm
- net BCLK_2: track 21.1 -> 22.3 mm
- net Jack_R: track 6.80 -> 7.41 mm
