File: 3_Technical_Documents/PCB/PM3_Audio_and_DMX_Template/PM3_Audio_and_DMX_Template/headphone_amp.kicad_sch (KiCad schematic)
At the start: 15 parts, among them U13 TPA6110A2DGN

Commit message: new push
Parts:
- renumbered C63 to C81, C64 to C82, C65 to C83, C66 to C84, C67 to C85, C68 to C86, C69 to C87, C70 to C88, C71 to C89, R70 to R62, R71 to R63, R72 to R64, R73 to R65, R74 to R66, U13 to U15
Changed lines of the file:
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@@
 		(dnp no)
 		(fields_autoplaced yes)
-		(property "Reference" "C68"
+		(property "Reference" "C86"
 			(at 177.8 57.1499 0)
 			(effects
@@
 			(project ""
 				(path "/1f276d59-ad9b-4e70-a842-f3b7e562eb9b/2329d9ea-d5d7-4913-84c5-e85a54af032e/8733e9e9-0235-42ab-8b67-3f0d5d49250e"
-					(reference "C68")
+					(reference "C86")
 					(unit 1)
 				)
@@
 		(on_board yes)
 		(dnp no)
-		(property "Reference" "R74"
+		(property "Reference" "R66"
 			(at 135.89 134.6199 0)
 			(effects
@@
 			(project ""
 				(path "/1f276d59-ad9b-4e70-a842-f3b7e562eb9b/2329d9ea-d5d7-4913-84c5-e85a54af032e/8733e9e9-0235-42ab-8b67-3f0d5d49250e"
-					(reference "R74")
+					(reference "R66")
 					(unit 1)
 				)
@@
 		(dnp no)
 		(fields_autoplaced yes)
-		(property "Reference" "#PWR096"
+		(property "Reference" "#PWR0114"
 			(at 168.91 121.92 0)
 			(effects
@@
 			(project ""
 				(path "/1f276d59-ad9b-4e70-a842-f3b7e562eb9b/2329d9ea-d5d7-4913-84c5-e85a54af032e/8733e9e9-0235-42ab-8b67-3f0d5d49250e"
-					(reference "#PWR096")
+					(reference "#PWR0114")
 					(unit 1)
 				)
@@
 		(dnp no)
 		(fields_autoplaced yes)
-		(property "Reference" "R70"
+		(property "Reference" "R62"
 			(at 101.6 82.55 90)
 			(effects
@@
 			(project ""
 				(path "/1f276d59-ad9b-4e70-a842-f3b7e562eb9b/2329d9ea-d5d7-4913-84c5-e85a54af032e/8733e9e9-0235-42ab-8b67-3f0d5d49250e"
-					(reference "R70")
+					(reference "R62")
 					(unit 1)
 				)
@@
 		(dnp no)
 		(fields_autoplaced yes)
-		(property "Reference" "#PWR097"
+		(property "Reference" "#PWR0115"
 			(at 173.99 76.2 0)
 			(effects
@@
 			(project ""
 				(path "/1f276d59-ad9b-4e70-a842-f3b7e562eb9b/2329d9ea-d5d7-4913-84c5-e85a54af032e/8733e9e9-0235-42ab-8b67-3f0d5d49250e"
-					(reference "#PWR097")
+					(reference "#PWR0115")
 					(unit 1)
 				)
@@
 		(dnp no)
 		(fields_autoplaced yes)
-		(property "Reference" "C65"
+		(property "Reference" "C83"
 			(at 124.46 77.4699 0)
 			(effects
@@
 			(project ""
 				(path "/1f276d59-ad9b-4e70-a842-f3b7e562eb9b/2329d9ea-d5d7-4913-84c5-e85a54af032e/8733e9e9-0235-42ab-8b67-3f0d5d49250e"
-					(reference "C65")
+					(reference "C83")
 					(unit 1)
 				)
@@
 		(on_board yes)
 		(dnp no)
-		(property "Reference" "C70"
+		(property "Reference" "C88"
 			(at 176.022 99.314 90)
 			(effects
@@
 			(project ""
 				(path "/1f276d59-ad9b-4e70-a842-f3b7e562eb9b/2329d9ea-d5d7-4913-84c5-e85a54af032e/8733e9e9-0235-42ab-8b67-3f0d5d49250e"
-					(reference "C70")
+					(reference "C88")
 					(unit 1)
 				)
@@
 		(on_board yes)
 		(dnp no)
-		(property "Reference" "C64"
+		(property "Reference" "C82"
 			(at 86.614 98.552 90)
 			(effects
@@
 			(project ""
 				(path "/1f276d59-ad9b-4e70-a842-f3b7e562eb9b/2329d9ea-d5d7-4913-84c5-e85a54af032e/8733e9e9-0235-42ab-8b67-3f0d5d49250e"
-					(reference "C64")
+					(reference "C82")
 					(unit 1)
 				)
@@
 		(on_board yes)
 		(dnp no)
-		(property "Reference" "R71"
+		(property "Reference" "R63"
 			(at 101.346 97.536 90)
 			(effects
@@
 			(project ""
 				(path "/1f276d59-ad9b-4e70-a842-f3b7e562eb9b/2329d9ea-d5d7-4913-84c5-e85a54af032e/8733e9e9-0235-42ab-8b67-3f0d5d49250e"
-					(reference "R71")
+					(reference "R63")
 					(unit 1)
 				)
@@
 		(dnp no)
 		(fields_autoplaced yes)
-		(property "Reference" "C69"
+		(property "Reference" "C87"
 			(at 174.371 81.28 90)
 			(effects
@@
 			(project ""
 				(path "/1f276d59-ad9b-4e70-a842-f3b7e562eb9b/2329d9ea-d5d7-4913-84c5-e85a54af032e/8733e9e9-0235-42ab-8b67-3f0d5d49250e"
-					(reference "C69")
+					(reference "C87")
 					(unit 1)
 				)
@@
 		(on_board yes)
 		(dnp no)
-		(property "Reference" "R72"
+		(property "Reference" "R64"
 			(at 113.03 77.4699 0)
 			(effects
@@
 			(project ""
 				(path "/1f276d59-ad9b-4e70-a842-f3b7e562eb9b/2329d9ea-d5d7-4913-84c5-e85a54af032e/8733e9e9-0235-42ab-8b67-3f0d5d49250e"
-					(reference "R72")
+					(reference "R64")
 					(unit 1)
 				)
@@
 		(dnp no)
 		(fields_autoplaced yes)
-		(property "Reference" "C66"
+		(property "Reference" "C84"
 			(at 124.46 111.7599 0)
 			(effects
@@
 			(project ""
 				(path "/1f276d59-ad9b-4e70-a842-f3b7e562eb9b/2329d9ea-d5d7-4913-84c5-e85a54af032e/8733e9e9-0235-42ab-8b67-3f0d5d49250e"
-					(reference "C66")
+					(reference "C84")
 					(unit 1)
 				)
@@
 		(on_board yes)
 		(dnp no)
-		(property "Reference" "R73"
+		(property "Reference" "R65"
 			(at 113.03 111.7599 0)
 			(effects
@@
 			(project ""
 				(path "/1f276d59-ad9b-4e70-a842-f3b7e562eb9b/2329d9ea-d5d7-4913-84c5-e85a54af032e/8733e9e9-0235-42ab-8b67-3f0d5d49250e"
-					(reference "R73")
+					(reference "R65")
 					(unit 1)
 				)
@@
 		(dnp no)
 		(fields_autoplaced yes)
-		(property "Reference" "U13"
+		(property "Reference" "U15"
 			(at 150.7333 78.74 0)
 			(effects
@@
 			(project ""
 				(path "/1f276d59-ad9b-4e70-a842-f3b7e562eb9b/2329d9ea-d5d7-4913-84c5-e85a54af032e/8733e9e9-0235-42ab-8b67-3f0d5d49250e"
-					(reference "U13")
+					(reference "U15")
 					(unit 1)
 				)
@@
 		(dnp no)
 		(fields_autoplaced yes)
-		(property "Reference" "#PWR094"
+		(property "Reference" "#PWR0112"
 			(at 148.59 48.26 0)
 			(effects
@@
 			(project ""
 				(path "/1f276d59-ad9b-4e70-a842-f3b7e562eb9b/2329d9ea-d5d7-4913-84c5-e85a54af032e/8733e9e9-0235-42ab-8b67-3f0d5d49250e"
-					(reference "#PWR094")
+					(reference "#PWR0112")
 					(unit 1)
 				)
@@
 		(dnp no)
 		(fields_autoplaced yes)
-		(property "Reference" "C71"
+		(property "Reference" "C89"
 			(at 189.23 56.2609 0)
 			(effects
@@
 			(project ""
 				(path "/1f276d59-ad9b-4e70-a842-f3b7e562eb9b/2329d9ea-d5d7-4913-84c5-e85a54af032e/8733e9e9-0235-42ab-8b67-3f0d5d49250e"
-					(reference "C71")
+					(reference "C89")
 					(unit 1)
 				)
@@
 		(dnp no)
 		(fields_autoplaced yes)
-		(property "Reference" "C67"
+		(property "Reference" "C85"
 			(at 172.72 107.9499 0)
 			(effects
@@
 			(project ""
 				(path "/1f276d59-ad9b-4e70-a842-f3b7e562eb9b/2329d9ea-d5d7-4913-84c5-e85a54af032e/8733e9e9-0235-42ab-8b67-3f0d5d49250e"
-					(reference "C67")
+					(reference "C85")
 					(unit 1)
 				)
@@
 		(dnp no)
 		(fields_autoplaced yes)
-		(property "Reference" "#PWR093"
+		(property "Reference" "#PWR0111"
 			(at 133.35 152.4 0)
 			(effects
@@
 			(project ""
 				(path "/1f276d59-ad9b-4e70-a842-f3b7e562eb9b/2329d9ea-d5d7-4913-84c5-e85a54af032e/8733e9e9-0235-42ab-8b67-3f0d5d49250e"
-					(reference "#PWR093")
+					(reference "#PWR0111")
 					(unit 1)
 				)
@@
 		(dnp no)
 		(fields_autoplaced yes)
-		(property "Reference" "#PWR095"
+		(property "Reference" "#PWR0113"
 			(at 148.59 118.11 0)
 			(effects
@@
 			(project ""
 				(path "/1f276d59-ad9b-4e70-a842-f3b7e562eb9b/2329d9ea-d5d7-4913-84c5-e85a54af032e/8733e9e9-0235-42ab-8b67-3f0d5d49250e"
-					(reference "#PWR095")
+					(reference "#PWR0113")
 					(unit 1)
 				)
@@
 		(dnp no)
 		(fields_autoplaced yes)
-		(property "Reference" "C63"
+		(property "Reference" "C81"
 			(at 87.249 81.28 90)
 			(effects
@@
 			(project ""
 				(path "/1f276d59-ad9b-4e70-a842-f3b7e562eb9b/2329d9ea-d5d7-4913-84c5-e85a54af032e/8733e9e9-0235-42ab-8b67-3f0d5d49250e"
-					(reference "C63")
-					(unit 1)
-				)
+					(reference "C81")
+					(unit 1)
+				)

Commit message: rework esp32, codec and layout
Parts:
- renumbered C81 to C66, C82 to C67, C83 to C68, C84 to C69, C85 to C70, C86 to C71, C87 to C72, C88 to C73, C89 to C74, R62 to R59, R63 to R60, R64 to R61, R65 to R62, R66 to R63, U15 to U14
Changed lines of the file:
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@@
 		(dnp no)
 		(fields_autoplaced yes)
-		(property "Reference" "C86"
+		(property "Reference" "C71"
 			(at 177.8 57.1499 0)
 			(effects
@@
 			(project ""
 				(path "/1f276d59-ad9b-4e70-a842-f3b7e562eb9b/2329d9ea-d5d7-4913-84c5-e85a54af032e/8733e9e9-0235-42ab-8b67-3f0d5d49250e"
-					(reference "C86")
+					(reference "C71")
 					(unit 1)
 				)
@@
 		(on_board yes)
 		(dnp no)
-		(property "Reference" "R66"
+		(property "Reference" "R63"
 			(at 135.89 134.6199 0)
 			(effects
@@
 			(project ""
 				(path "/1f276d59-ad9b-4e70-a842-f3b7e562eb9b/2329d9ea-d5d7-4913-84c5-e85a54af032e/8733e9e9-0235-42ab-8b67-3f0d5d49250e"
-					(reference "R66")
+					(reference "R63")
 					(unit 1)
 				)
@@
 		(dnp no)
 		(fields_autoplaced yes)
-		(property "Reference" "#PWR0114"
+		(property "Reference" "#PWR0103"
 			(at 168.91 121.92 0)
 			(effects
@@
 			(project ""
 				(path "/1f276d59-ad9b-4e70-a842-f3b7e562eb9b/2329d9ea-d5d7-4913-84c5-e85a54af032e/8733e9e9-0235-42ab-8b67-3f0d5d49250e"
-					(reference "#PWR0114")
+					(reference "#PWR0103")
 					(unit 1)
 				)
@@
 		(dnp no)
 		(fields_autoplaced yes)
-		(property "Reference" "R62"
+		(property "Reference" "R59"
 			(at 101.6 82.55 90)
 			(effects
@@
 			(project ""
 				(path "/1f276d59-ad9b-4e70-a842-f3b7e562eb9b/2329d9ea-d5d7-4913-84c5-e85a54af032e/8733e9e9-0235-42ab-8b67-3f0d5d49250e"
-					(reference "R62")
+					(reference "R59")
 					(unit 1)
 				)
@@
 		(dnp no)
 		(fields_autoplaced yes)
-		(property "Reference" "#PWR0115"
+		(property "Reference" "#PWR0104"
 			(at 173.99 76.2 0)
 			(effects
@@
 			(project ""
 				(path "/1f276d59-ad9b-4e70-a842-f3b7e562eb9b/2329d9ea-d5d7-4913-84c5-e85a54af032e/8733e9e9-0235-42ab-8b67-3f0d5d49250e"
-					(reference "#PWR0115")
+					(reference "#PWR0104")
 					(unit 1)
 				)
@@
 		(dnp no)
 		(fields_autoplaced yes)
-		(property "Reference" "C83"
+		(property "Reference" "C68"
 			(at 124.46 77.4699 0)
 			(effects
@@
 			(project ""
 				(path "/1f276d59-ad9b-4e70-a842-f3b7e562eb9b/2329d9ea-d5d7-4913-84c5-e85a54af032e/8733e9e9-0235-42ab-8b67-3f0d5d49250e"
-					(reference "C83")
+					(reference "C68")
 					(unit 1)
 				)
@@
 		(on_board yes)
 		(dnp no)
-		(property "Reference" "C88"
+		(property "Reference" "C73"
 			(at 176.022 99.314 90)
 			(effects
@@
 			(project ""
 				(path "/1f276d59-ad9b-4e70-a842-f3b7e562eb9b/2329d9ea-d5d7-4913-84c5-e85a54af032e/8733e9e9-0235-42ab-8b67-3f0d5d49250e"
-					(reference "C88")
+					(reference "C73")
 					(unit 1)
 				)
@@
 		(on_board yes)
 		(dnp no)
-		(property "Reference" "C82"
+		(property "Reference" "C67"
 			(at 86.614 98.552 90)
 			(effects
@@
 			(project ""
 				(path "/1f276d59-ad9b-4e70-a842-f3b7e562eb9b/2329d9ea-d5d7-4913-84c5-e85a54af032e/8733e9e9-0235-42ab-8b67-3f0d5d49250e"
-					(reference "C82")
+					(reference "C67")
 					(unit 1)
 				)
@@
 		(on_board yes)
 		(dnp no)
-		(property "Reference" "R63"
+		(property "Reference" "R60"
 			(at 101.346 97.536 90)
 			(effects
@@
 			(project ""
 				(path "/1f276d59-ad9b-4e70-a842-f3b7e562eb9b/2329d9ea-d5d7-4913-84c5-e85a54af032e/8733e9e9-0235-42ab-8b67-3f0d5d49250e"
-					(reference "R63")
+					(reference "R60")
 					(unit 1)
 				)
@@
 		(dnp no)
 		(fields_autoplaced yes)
-		(property "Reference" "C87"
+		(property "Reference" "C72"
 			(at 174.371 81.28 90)
 			(effects
@@
 			(project ""
 				(path "/1f276d59-ad9b-4e70-a842-f3b7e562eb9b/2329d9ea-d5d7-4913-84c5-e85a54af032e/8733e9e9-0235-42ab-8b67-3f0d5d49250e"
-					(reference "C87")
+					(reference "C72")
 					(unit 1)
 				)
@@
 		(on_board yes)
 		(dnp no)
-		(property "Reference" "R64"
+		(property "Reference" "R61"
 			(at 113.03 77.4699 0)
 			(effects
@@
 			(project ""
 				(path "/1f276d59-ad9b-4e70-a842-f3b7e562eb9b/2329d9ea-d5d7-4913-84c5-e85a54af032e/8733e9e9-0235-42ab-8b67-3f0d5d49250e"
-					(reference "R64")
+					(reference "R61")
 					(unit 1)
 				)
@@
 		(dnp no)
 		(fields_autoplaced yes)
-		(property "Reference" "C84"
+		(property "Reference" "C69"
 			(at 124.46 111.7599 0)
 			(effects
@@
 			(project ""
 				(path "/1f276d59-ad9b-4e70-a842-f3b7e562eb9b/2329d9ea-d5d7-4913-84c5-e85a54af032e/8733e9e9-0235-42ab-8b67-3f0d5d49250e"
-					(reference "C84")
+					(reference "C69")
 					(unit 1)
 				)
@@
 		(on_board yes)
 		(dnp no)
-		(property "Reference" "R65"
+		(property "Reference" "R62"
 			(at 113.03 111.7599 0)
 			(effects
@@
 			(project ""
 				(path "/1f276d59-ad9b-4e70-a842-f3b7e562eb9b/2329d9ea-d5d7-4913-84c5-e85a54af032e/8733e9e9-0235-42ab-8b67-3f0d5d49250e"
-					(reference "R65")
+					(reference "R62")
 					(unit 1)
 				)
@@
 		(dnp no)
 		(fields_autoplaced yes)
-		(property "Reference" "U15"
+		(property "Reference" "U14"
 			(at 150.7333 78.74 0)
 			(effects
@@
 			(project ""
 				(path "/1f276d59-ad9b-4e70-a842-f3b7e562eb9b/2329d9ea-d5d7-4913-84c5-e85a54af032e/8733e9e9-0235-42ab-8b67-3f0d5d49250e"
-					(reference "U15")
+					(reference "U14")
 					(unit 1)
 				)
@@
 		(dnp no)
 		(fields_autoplaced yes)
-		(property "Reference" "#PWR0112"
+		(property "Reference" "#PWR0101"
 			(at 148.59 48.26 0)
 			(effects
@@
 			(project ""
 				(path "/1f276d59-ad9b-4e70-a842-f3b7e562eb9b/2329d9ea-d5d7-4913-84c5-e85a54af032e/8733e9e9-0235-42ab-8b67-3f0d5d49250e"
-					(reference "#PWR0112")
+					(reference "#PWR0101")
 					(unit 1)
 				)
@@
 		(dnp no)
 		(fields_autoplaced yes)
-		(property "Reference" "C89"
+		(property "Reference" "C74"
 			(at 189.23 56.2609 0)
 			(effects
@@
 			(project ""
 				(path "/1f276d59-ad9b-4e70-a842-f3b7e562eb9b/2329d9ea-d5d7-4913-84c5-e85a54af032e/8733e9e9-0235-42ab-8b67-3f0d5d49250e"
-					(reference "C89")
+					(reference "C74")
 					(unit 1)
 				)
@@
 		(dnp no)
 		(fields_autoplaced yes)
-		(property "Reference" "C85"
+		(property "Reference" "C70"
 			(at 172.72 107.9499 0)
 			(effects
@@
 			(project ""
 				(path "/1f276d59-ad9b-4e70-a842-f3b7e562eb9b/2329d9ea-d5d7-4913-84c5-e85a54af032e/8733e9e9-0235-42ab-8b67-3f0d5d49250e"
-					(reference "C85")
+					(reference "C70")
 					(unit 1)
 				)
@@
 		(dnp no)
 		(fields_autoplaced yes)
-		(property "Reference" "#PWR0111"
+		(property "Reference" "#PWR0100"
 			(at 133.35 152.4 0)
 			(effects
@@
 			(project ""
 				(path "/1f276d59-ad9b-4e70-a842-f3b7e562eb9b/2329d9ea-d5d7-4913-84c5-e85a54af032e/8733e9e9-0235-42ab-8b67-3f0d5d49250e"
-					(reference "#PWR0111")
+					(reference "#PWR0100")
 					(unit 1)
 				)
@@
 		(dnp no)
 		(fields_autoplaced yes)
-		(property "Reference" "#PWR0113"
+		(property "Reference" "#PWR0102"
 			(at 148.59 118.11 0)
 			(effects
@@
 			(project ""
 				(path "/1f276d59-ad9b-4e70-a842-f3b7e562eb9b/2329d9ea-d5d7-4913-84c5-e85a54af032e/8733e9e9-0235-42ab-8b67-3f0d5d49250e"
-					(reference "#PWR0113")
+					(reference "#PWR0102")
 					(unit 1)
 				)
@@
 		(dnp no)
 		(fields_autoplaced yes)
-		(property "Reference" "C81"
+		(property "Reference" "C66"
 			(at 87.249 81.28 90)
 			(effects
@@
 			(project ""
 				(path "/1f276d59-ad9b-4e70-a842-f3b7e562eb9b/2329d9ea-d5d7-4913-84c5-e85a54af032e/8733e9e9-0235-42ab-8b67-3f0d5d49250e"
-					(reference "C81")
-					(unit 1)
-				)
+					(reference "C66")
+					(unit 1)
+				)

Commit message: schematics, layout and bom updated (to match corrections)
Parts:
- C70: value 1u CER -> 1u
Changed lines of the file:
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@@
 			)
 		)
-		(property "Value" "1u CER"
+		(property "Value" "1u"
 			(at 172.72 110.4899 0)
 			(effects
