File: 3_Technical_Documents/PCB/PM3_Audio_and_DMX_Template/PM3_Audio_and_DMX_Template/codec_and_buffers.kicad_sch (KiCad schematic)
At the start: 19 parts, among them U9 CS4271

Commit message: new push
Parts:
- removed C30: 100n, Capacitor_SMD:C_0603_1608Metric, symbol Device:C
- removed C31: 1u, Capacitor_SMD:C_0805_2012Metric, symbol Device:C
- removed C41: 47u, Capacitor_SMD:CP_Elec_6.3x7.7, symbol Device:C_Polarized
- removed R17, R33: 10k, Resistor_SMD:R_0603_1608Metric, symbol Device:R
- added R29, R30, R32, R35: 10k, Resistor_SMD:R_0603_1608Metric, symbol Device:R
- added R31: 47k, Resistor_SMD:R_0603_1608Metric, symbol Device:R
- renumbered C13 to C30, C14 to C31, C33 to C35, C34 to C36, C35 to C37, C36 to C38, C37 to C39, C15 to C40, C17 to C41, C38 to C42, C16 to C43, C32 to C44, U9 to U10
Connections:
- net +3.3V: now also C37.1, C38.1, U10.9 (VD)
- net +3V0: now also C35.1, C36.1, U10.10 (VL), R29.2, R30.2, R31.2
- net +5VA: no longer C35.1, C36.1, C37.1, C38.1, U10.10 (VL), U10.9 (VD)
- net CODEC_SCL: now also R30.1, R32.2
- net CODEC_SDA: now also R29.1, R35.2
- net GND: now also R32.1, R35.1
- net SDOUT: now also R31.1

Commit message: codec and layout
Parts:
- added R36, R39, R40, R43: 22R, Resistor_SMD:R_0603_1608Metric, symbol Device:R
Connections:
- net +3V0: now also U10.23 (~{AMUTEC}), U10.28 (~{BMUTEC})
- net GND: now also U10.13 (AD0/~{CS}(I2S/~{LJ}))
- net LRCK: now also R40.2; no longer U10.4 (LRCK)
- net MCLK: now also R43.1; no longer U10.3 (MCLK)
- net SCLK: now also R39.2; no longer U10.5 (SCLK)
- net SDIN: now also R36.2; no longer U10.7 (SDIN)
- new net: R40.1, U10.4 (LRCK)
- new net: R39.1, U10.5 (SCLK)
- new net: R36.1, U10.7 (SDIN)
- new net: R43.2, U10.3 (MCLK)

Commit message: rework esp32, codec and layout
Parts:
- renumbered C35 to C32, C36 to C33, C37 to C34, C38 to C35, C39 to C36, C40 to C37, C41 to C38, C42 to C39, C43 to C40, C44 to C41, R30 to R28, R32 to R29, R29 to R30, R35 to R31, R31 to R32, R43 to R33, R40 to R34, R39 to R35

Commit message: esp-stm connection (+ conflict recolution)
Parts:
- added R4: 10k, Resistor_SMD:R_0603_1608Metric, symbol Device:R
Connections:
- net +3V0: now also R4.1
- net GND: no longer U10.13 (AD0/~{CS}(I2S/~{LJ}))
- new net: R4.2, U10.13 (AD0/~{CS}(I2S/~{LJ}))
Changed lines of the file:
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@@
 	(wire
 		(pts
+			(xy 120.65 113.03) (xy 120.65 114.3)
+		)
+		(stroke
+			(width 0)
+			(type default)
+		)
+	)
+	(wire
+		(pts
 			(xy 222.25 134.62) (xy 228.6 134.62)
 		)
@@
 	(wire
 		(pts
+			(xy 116.84 121.92) (xy 120.65 121.92)
+		)
+		(stroke
+			(width 0)
+			(type default)
+		)
+	)
+	(wire
+		(pts
 			(xy 34.29 149.86) (xy 29.21 149.86)
 		)
@@
 	(wire
 		(pts
-			(xy 124.46 113.03) (xy 127 113.03)
-		)
-		(stroke
-			(width 0)
-			(type default)
-		)
-	)
-	(wire
-		(pts
 			(xy 168.91 33.02) (xy 175.26 33.02)
 		)
@@
 	(wire
 		(pts
+			(xy 120.65 113.03) (xy 127 113.03)
+		)
+		(stroke
+			(width 0)
+			(type default)
+		)
+	)
+	(wire
+		(pts
 			(xy 228.6 134.62) (xy 228.6 107.95)
 		)
@@
 	(wire
 		(pts
-			(xy 124.46 115.57) (xy 124.46 113.03)
-		)
-		(stroke
-			(width 0)
-			(type default)
-		)
-	)
-	(wire
-		(pts
 			(xy 172.72 60.96) (xy 186.69 60.96)
 		)
@@
 	)
 	(symbol
-		(lib_id "power:GND")
-		(at 124.46 115.57 0)
-		(unit 1)
-		(exclude_from_sim no)
-		(in_bom yes)
-		(on_board yes)
-		(dnp no)
-		(fields_autoplaced yes)
-		(property "Reference" "#PWR077"
-			(at 124.46 121.92 0)
-			(effects
-				(font
-					(size 1.27 1.27)
-				)
-				(hide yes)
-			)
-		)
-		(property "Value" "GND"
-			(at 124.46 120.65 0)
-			(effects
-				(font
-					(size 1.27 1.27)
-				)
-			)
-		)
-		(property "Footprint" ""
-			(at 124.46 115.57 0)
-			(effects
-				(font
-					(size 1.27 1.27)
-				)
-				(hide yes)
-			)
-		)
-		(property "Datasheet" ""
-			(at 124.46 115.57 0)
-			(effects
-				(font
-					(size 1.27 1.27)
-				)
-				(hide yes)
-			)
-		)
-		(property "Description" "Power symbol creates a global label with name \"GND\" , ground"
-			(at 124.46 115.57 0)
-			(effects
-				(font
-					(size 1.27 1.27)
-				)
-				(hide yes)
-			)
-		)
-		(pin "1"
-		)
-		(instances
-			(project "PM3_Audio_and_DMX"
-				(path "/1f276d59-ad9b-4e70-a842-f3b7e562eb9b/2329d9ea-d5d7-4913-84c5-e85a54af032e/5f71fd42-8f86-4900-bb58-dbcd17a8cc2c"
-					(reference "#PWR077")
-					(unit 1)
-				)
-			)
-		)
-	)
-	(symbol
 		(lib_id "Device:C")
 		(at 172.72 68.58 0)
@@
 	)
 	(symbol
+		(lib_id "power:+3V0")
+		(at 116.84 121.92 0)
+		(unit 1)
+		(exclude_from_sim no)
+		(in_bom yes)
+		(on_board yes)
+		(dnp no)
+		(property "Reference" "#PWR022"
+			(at 116.84 125.73 0)
+			(effects
+				(font
+					(size 1.27 1.27)
+				)
+				(hide yes)
+			)
+		)
+		(property "Value" "+3V0"
+			(at 116.84 116.84 90)
+			(effects
+				(font
+					(size 1.27 1.27)
+				)
+			)
+		)
+		(property "Footprint" ""
+			(at 116.84 121.92 0)
+			(effects
+				(font
+					(size 1.27 1.27)
+				)
+				(hide yes)
+			)
+		)
+		(property "Datasheet" ""
+			(at 116.84 121.92 0)
+			(effects
+				(font
+					(size 1.27 1.27)
+				)
+				(hide yes)
+			)
+		)
+		(property "Description" "Power symbol creates a global label with name \"+3V0\""
+			(at 116.84 121.92 0)
+			(effects
+				(font
+					(size 1.27 1.27)
+				)
+				(hide yes)
+			)
+		)
+		(pin "1"
+		)
+		(instances
+			(project "PM3_Audio_and_DMX"
+				(path "/1f276d59-ad9b-4e70-a842-f3b7e562eb9b/2329d9ea-d5d7-4913-84c5-e85a54af032e/5f71fd42-8f86-4900-bb58-dbcd17a8cc2c"
+					(reference "#PWR022")
+					(unit 1)
+				)
+			)
+		)
+	)
+	(symbol
 		(lib_id "Device:C")
 		(at 180.34 27.94 0)
@@
 					(unit 1)
 				)
+			)
+		)
+	)
+	(symbol
+		(lib_id "Device:R")
+		(at 120.65 118.11 180)
+		(unit 1)
+		(exclude_from_sim no)
+		(in_bom yes)
+		(on_board yes)
+		(dnp no)
+		(fields_autoplaced yes)
+		(property "Reference" "R4"
+			(at 123.19 116.8399 0)
+			(effects
+				(font
+					(size 1.27 1.27)
+				)
+				(justify right)
+			)
+		)
+		(property "Value" "10k"
+			(at 123.19 119.3799 0)
+			(effects
+				(font
+					(size 1.27 1.27)
+				)
+				(justify right)
+			)
+		)
+		(property "Footprint" "Resistor_SMD:R_0603_1608Metric"
+			(at 122.428 118.11 90)
+			(effects
+				(font
+					(size 1.27 1.27)
+				)
+				(hide yes)
+			)
+		)
+		(property "Datasheet" "~"
+			(at 120.65 118.11 0)
+			(effects
+				(font
+					(size 1.27 1.27)
+				)
+				(hide yes)
+			)
+		)
+		(property "Description" "Resistor"
+			(at 120.65 118.11 0)
+			(effects
+				(font
+					(size 1.27 1.27)
+				)
+				(hide yes)
+			)
+		)
+		(property "MPN" "GPR060310K"
+			(at 120.65 118.11 0)
+			(effects
+				(font
+					(size 1.27 1.27)
+				)
+				(hide yes)
+			)
+		)
+		(property "Manufacturer" ""
+			(at 120.65 118.11 0)
+			(effects
+				(font
+					(size 1.27 1.27)
+				)
+				(hide yes)
+			)
+		)
+		(pin "1"
+		)
+		(pin "2"
+		)
+		(instances
+			(project "PM3_Audio_and_DMX"
+				(path "/1f276d59-ad9b-4e70-a842-f3b7e562eb9b/2329d9ea-d5d7-4913-84c5-e85a54af032e/5f71fd42-8f86-4900-bb58-dbcd17a8cc2c"
+					(reference "R4")
+					(unit 1)
+				)

Commit message: Amutec und Bmutec left floating
Connections:
- net +3V0: no longer U10.23 (~{AMUTEC}), U10.28 (~{BMUTEC})
- no-connect marks 0 -> 2
Changed lines of the file:
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@@
-	)
-	(junction
-		(at 158.75 85.09)
-		(diameter 0)
-		(color 0 0 0 0)
 	)
 	(junction
@@
 		(color 0 0 0 0)
 	)
+	(no_connect
+		(at 157.48 85.09)
+	)
+	(no_connect
+		(at 157.48 87.63)
+	)
 	(wire
 		(pts
@@
 	(wire
 		(pts
-			(xy 158.75 71.12) (xy 158.75 85.09)
-		)
-		(stroke
-			(width 0)
-			(type default)
-		)
-	)
-	(wire
-		(pts
 			(xy 226.06 139.7) (xy 226.06 113.03)
 		)
@@
 	(wire
 		(pts
-			(xy 158.75 85.09) (xy 158.75 87.63)
-		)
-		(stroke
-			(width 0)
-			(type default)
-		)
-	)
-	(wire
-		(pts
 			(xy 123.19 90.17) (xy 127 90.17)
 		)
@@
 	(wire
 		(pts
-			(xy 157.48 85.09) (xy 158.75 85.09)
-		)
-		(stroke
-			(width 0)
-			(type default)
-		)
-	)
-	(wire
-		(pts
 			(xy 123.19 92.71) (xy 127 92.71)
 		)
@@
 		(pts
 			(xy 157.48 80.01) (xy 162.56 80.01)
-		)
-		(stroke
-			(width 0)
-			(type default)
-		)
-	)
-	(wire
-		(pts
-			(xy 158.75 87.63) (xy 157.48 87.63)
 		)
 		(stroke
@@
 			(effects
 				(font
-					(size 1.27 1.27)
-				)
-				(justify left)
-				(hide yes)
-			)
-		)
-	)
-	(global_label "VL"
-		(shape input)
-		(at 158.75 71.12 90)
-		(fields_autoplaced yes)
-		(effects
-			(font
-				(size 1.016 1.016)
-			)
-			(justify left)
-		)
-		(property "Intersheetrefs" "${INTERSHEET_REFS}"
-			(at 158.75 67.0387 90)
-			(effects
-				(font

Commit message: reqorked pcb
Parts:
- added R64: 10k, Resistor_SMD:R_0603_1608Metric, symbol Device:R
Connections:
- net +3V0: now also R64.2
- net CODEC_RESETN: now also R64.1
Changed lines of the file:
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@@
+	)
+	(junction
+		(at 120.65 77.47)
+		(diameter 0)
+		(color 0 0 0 0)
 	)
 	(junction
@@
 	(wire
 		(pts
+			(xy 120.65 74.93) (xy 120.65 77.47)
+		)
+		(stroke
+			(width 0)
+			(type default)
+		)
+	)
+	(wire
+		(pts
 			(xy 157.48 97.79) (xy 208.28 97.79)
 		)
@@
 	(wire
 		(pts
-			(xy 110.49 77.47) (xy 127 77.47)
+			(xy 110.49 77.47) (xy 120.65 77.47)
 		)
 		(stroke
@@
 	(wire
 		(pts
+			(xy 120.65 77.47) (xy 127 77.47)
+		)
+		(stroke
+			(width 0)
+			(type default)
+		)
+	)
+	(wire
+		(pts
 			(xy 123.19 90.17) (xy 127 90.17)
 		)
@@
 		(pts
 			(xy 153.67 21.59) (xy 153.67 24.13)
+		)
+		(stroke
+			(width 0)
+			(type default)
+		)
+	)
+	(wire
+		(pts
+			(xy 120.65 64.77) (xy 120.65 67.31)
 		)
 		(stroke
@@
 				)
 				(justify right)
+				(hide yes)
+			)
+		)
+	)
+	(global_label "VL"
+		(shape input)
+		(at 120.65 64.77 90)
+		(fields_autoplaced yes)
+		(effects
+			(font
+				(size 1.016 1.016)
+			)
+			(justify left)
+		)
+		(property "Intersheetrefs" "${INTERSHEET_REFS}"
+			(at 120.65 60.6887 90)
+			(effects
+				(font
+					(size 1.27 1.27)
+				)
+				(justify left)
 				(hide yes)
 			)
@@
 					(unit 1)
 				)
+			)
+		)
+	)
+	(symbol
+		(lib_id "Device:R")
+		(at 120.65 71.12 180)
+		(unit 1)
+		(exclude_from_sim no)
+		(in_bom yes)
+		(on_board yes)
+		(dnp no)
+		(fields_autoplaced yes)
+		(property "Reference" "R64"
+			(at 123.19 69.8499 0)
+			(effects
+				(font
+					(size 1.27 1.27)
+				)
+				(justify right)
+			)
+		)
+		(property "Value" "10k"
+			(at 123.19 72.3899 0)
+			(effects
+				(font
+					(size 1.27 1.27)
+				)
+				(justify right)
+			)
+		)
+		(property "Footprint" "Resistor_SMD:R_0603_1608Metric"
+			(at 122.428 71.12 90)
+			(effects
+				(font
+					(size 1.27 1.27)
+				)
+				(hide yes)
+			)
+		)
+		(property "Datasheet" "~"
+			(at 120.65 71.12 0)
+			(effects
+				(font
+					(size 1.27 1.27)
+				)
+				(hide yes)
+			)
+		)
+		(property "Description" "Resistor"
+			(at 120.65 71.12 0)
+			(effects
+				(font
+					(size 1.27 1.27)
+				)
+				(hide yes)
+			)
+		)
+		(property "MPN" "GPR060310K"
+			(at 120.65 71.12 0)
+			(effects
+				(font
+					(size 1.27 1.27)
+				)
+				(hide yes)
+			)
+		)
+		(property "Manufacturer" ""
+			(at 120.65 71.12 0)
+			(effects
+				(font
+					(size 1.27 1.27)
+				)
+				(hide yes)
+			)
+		)
+		(property "Sim.Type" ""
+			(at 120.65 71.12 0)
+			(effects
+				(font
+					(size 1.27 1.27)
+				)
+				(hide yes)
+			)
+		)
+		(pin "1"
+		)
+		(pin "2"
+		)
+		(instances
+			(project "PM3_Audio_and_DMX"
+				(path "/1f276d59-ad9b-4e70-a842-f3b7e562eb9b/2329d9ea-d5d7-4913-84c5-e85a54af032e/5f71fd42-8f86-4900-bb58-dbcd17a8cc2c"
+					(reference "R64")
+					(unit 1)
+				)

Commit message: comments in schematics
Other:
- note added: "R29 dnp"
- note added: "R30 dnp"
Changed lines of the file:
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@@
 	(generator_version "9.0")
 	(paper "A4")
+	(text "R30 dnp"
+		(exclude_from_sim no)
+		(at 78.994 104.14 0)
+		(effects
+			(font
+				(size 1.27 1.27)
+				(color 255 0 0 1)
+			)
+		)
+	)
+	(text "R29 dnp"
+		(exclude_from_sim no)
+		(at 58.928 113.284 0)
+		(effects
+			(font
+				(size 1.27 1.27)
+				(color 255 0 0 1)
+			)
+		)
+	)
 	(junction
 		(at 148.59 33.02)
@@
 		)
 		(property "Value" "+3V0"
-			(at 121.92 15.24 90)
-			(effects
-				(font
+			(at 121.92 15.24 0)
+			(effects
+				(font
